Commit message: added stepper interface

File: src/nick_bot/description/OG/robot_core.xacro (robot description, xacro)
@@ -2,27 +2,43 @@
 <robot xmlns:xacro="http://www.ros.org/wiki/xacro">
   <xacro:property name="joint_damping" value="1.0"/>
+  <link name="world"/>
+  <joint name="base_joint" type="fixed">
+    <parent link="world"/>
+    <child link="base_link"/>
+    <origin rpy="0 0 0" xyz="0.0 0.0 0.3"/>
+  </joint>
   <link
     name="base_link">
-    <visual>
-      <origin
-        xyz="0 0 0"
-        rpy="0 0 0" />
-      <geometry>
-        <mesh
-          filename="package://nick_bot_1/meshes/base_link.STL" />
-      </geometry>
-      <material
-        name="">
-        <color
-          rgba="0.79216 0.81961 0.93333 1" />
-      </material>
-    </visual>
-    <collision>
-      <origin
-        xyz="0 0 0"
-        rpy="0 0 0" />
-      <geometry>
-        <mesh
-          filename="package://nick_bot_1/meshes/base_link.STL" />
+    <inertial>
+      <origin
+        xyz="0 0 2"
+        rpy="0 0 0" />
+      <mass
+        value="0.05" />
+      <inertia ixx="0.0001" ixy="0.000"  ixz="0.000"
+         iyy="0.0001" iyz="0.000"
+         izz="0.0001"/>
+    </inertial>
+    <visual>
+      <origin
+        xyz="0 0 0"
+        rpy="0 0 0" />
+      <geometry>
+        <mesh
+          filename="package://nick_bot/meshes/base_link.STL" />
+      </geometry>
+      <material
+        name="">
+        <color
+          rgba="0.79216 0.81961 0.93333 1" />
+      </material>
+    </visual>
+    <collision>
+      <origin
+        xyz="0 0 0"
+        rpy="0 0 0" />
+      <geometry>
+        <mesh
+          filename="package://nick_bot/meshes/base_link.STL" />
       </geometry>
     </collision>
@@ -35,34 +51,30 @@
         rpy="0 0 0" />
       <mass
-        value="0.28024" />
-      <inertia
-        ixx="0.00026699"
-        ixy="1.8167E-07"
-        ixz="2.7958E-05"
-        iyy="0.00023186"
-        iyz="-1.865E-06"
-        izz="0.00013903" />
-    </inertial>
-    <visual>
-      <origin
-        xyz="0 0 0"
-        rpy="0 0 0" />
-      <geometry>
-        <mesh
-          filename="package://nick_bot_1/meshes/link_1.STL" />
-      </geometry>
-      <material
-        name="">
-        <color
-          rgba="0.79216 0.81961 0.93333 1" />
-      </material>
-    </visual>
-    <collision>
-      <origin
-        xyz="0 0 0"
-        rpy="0 0 0" />
-      <geometry>
-        <mesh
-          filename="package://nick_bot_1/meshes/link_1.STL" />
+        value="0.05" />
+      <inertia ixx="0.0001" ixy="0.000"  ixz="0.000"
+         iyy="0.0001" iyz="0.000"
+         izz="0.0001"/>
+    </inertial>
+    <visual>
+      <origin
+        xyz="0 0 0"
+        rpy="0 0 0" />
+      <geometry>
+        <mesh
+          filename="package://nick_bot/meshes/link_1.STL" />
+      </geometry>
+      <material
+        name="">
+        <color
+          rgba="0.79216 0.81961 0.93333 1" />
+      </material>
+    </visual>
+    <collision>
+      <origin
+        xyz="0 0 0"
+        rpy="0 0 0" />
+      <geometry>
+        <mesh
+          filename="package://nick_bot/meshes/link_1.STL" />
       </geometry>
     </collision>
@@ -83,7 +95,6 @@
       lower="-2.7"
       upper="2.7"
-      effort="300"
-      velocity="4" />
-    <dynamics damping="${joint_damping}"/>
+      effort="300.0"
+      velocity="4.0" />
   </joint>
   <link
@@ -94,34 +105,30 @@
         rpy="0 0 0" />
       <mass
-        value="0.29393" />
-      <inertia
-        ixx="0.00033457"
-        ixy="-6.6415E-07"
-        ixz="-3.3309E-05"
-        iyy="0.00032504"
-        iyz="-3.5156E-06"
-        izz="0.00010703" />
-    </inertial>
-    <visual>
-      <origin
-        xyz="0 0 0"
-        rpy="0 0 0" />
-      <geometry>
-        <mesh
-          filename="package://nick_bot_1/meshes/link_2.STL" />
-      </geometry>
-      <material
-        name="">
-        <color
-          rgba="0.79216 0.81961 0.93333 1" />
-      </material>
-    </visual>
-    <collision>
-      <origin
-        xyz="0 0 0"
-        rpy="0 0 0" />
-      <geometry>
-        <mesh
-          filename="package://nick_bot_1/meshes/link_2.STL" />
+        value="0.05" />
+      <inertia ixx="0.0001" ixy="0.000"  ixz="0.000"
+         iyy="0.0001" iyz="0.000"
+         izz="0.0001"/>
+    </inertial>
+    <visual>
+      <origin
+        xyz="0 0 0"
+        rpy="0 0 0" />
+      <geometry>
+        <mesh
+          filename="package://nick_bot/meshes/link_2.STL" />
+      </geometry>
+      <material
+        name="">
+        <color
+          rgba="0.79216 0.81961 0.93333 1" />
+      </material>
+    </visual>
+    <collision>
+      <origin
+        xyz="0 0 0"
+        rpy="0 0 0" />
+      <geometry>
+        <mesh
+          filename="package://nick_bot/meshes/link_2.STL" />
       </geometry>
     </collision>
@@ -143,6 +150,5 @@
       upper="0.6"
       effort="300"
-      velocity="4" />
-    <dynamics damping="${joint_damping}"/>
+      velocity="4.0" />
   </joint>
   <link
@@ -153,34 +159,30 @@
         rpy="0 0 0" />
       <mass
-        value="0.085607" />
-      <inertia
-        ixx="5.4273E-05"
-        ixy="-3.1645E-08"
-        ixz="7.4467E-07"
-        iyy="4.5008E-05"
-        iyz="-2.8453E-07"
-        izz="3.1724E-05" />
-    </inertial>
-    <visual>
-      <origin
-        xyz="0 0 0"
-        rpy="0 0 0" />
-      <geometry>
-        <mesh
-          filename="package://nick_bot_1/meshes/link_3.STL" />
-      </geometry>
-      <material
-        name="">
-        <color
-          rgba="0.79216 0.81961 0.93333 1" />
-      </material>
-    </visual>
-    <collision>
-      <origin
-        xyz="0 0 0"
-        rpy="0 0 0" />
-      <geometry>
-        <mesh
-          filename="package://nick_bot_1/meshes/link_3.STL" />
+        value="0.05" />
+      <inertia ixx="0.0001" ixy="0.000"  ixz="0.000"
+         iyy="0.0001" iyz="0.000"
+         izz="0.0001"/>
+    </inertial>
+    <visual>
+      <origin
+        xyz="0 0 0"
+        rpy="0 0 0" />
+      <geometry>
+        <mesh
+          filename="package://nick_bot/meshes/link_3.STL" />
+      </geometry>
+      <material
+        name="">
+        <color
+          rgba="0.79216 0.81961 0.93333 1" />
+      </material>
+    </visual>
+    <collision>
+      <origin
+        xyz="0 0 0"
+        rpy="0 0 0" />
+      <geometry>
+        <mesh
+          filename="package://nick_bot/meshes/link_3.STL" />
       </geometry>
     </collision>
@@ -202,6 +204,5 @@
       upper="4"
       effort="200"
-      velocity="4" />
-    <dynamics damping="${joint_damping}"/>
+      velocity="4.0" />
   </joint>
   <link
@@ -212,34 +213,30 @@
         rpy="0 0 0" />
       <mass
-        value="0.15698" />
-      <inertia
-        ixx="0.0003485"
-        ixy="3.586E-08"
-        ixz="-7.8887E-07"
-        iyy="0.00035409"
-        iyz="-5.1436E-06"
-        izz="5.9114E-05" />
-    </inertial>
-    <visual>
-      <origin
-        xyz="0 0 0"
-        rpy="0 0 0" />
-      <geometry>
-        <mesh
-          filename="package://nick_bot_1/meshes/link_4.STL" />
-      </geometry>
-      <material
-        name="">
-        <color
-          rgba="0.79216 0.81961 0.93333 1" />
-      </material>
-    </visual>
-    <collision>
-      <origin
-        xyz="0 0 0"
-        rpy="0 0 0" />
-      <geometry>
-        <mesh
-          filename="package://nick_bot_1/meshes/link_4.STL" />
+        value="0.05" />
+      <inertia ixx="0.0001" ixy="0.000"  ixz="0.000"
+         iyy="0.0001" iyz="0.000"
+         izz="0.0001"/>
+    </inertial>
+    <visual>
+      <origin
+        xyz="0 0 0"
+        rpy="0 0 0" />
+      <geometry>
+        <mesh
+          filename="package://nick_bot/meshes/link_4.STL" />
+      </geometry>
+      <material
+        name="">
+        <color
+          rgba="0.79216 0.81961 0.93333 1" />
+      </material>
+    </visual>
+    <collision>
+      <origin
+        xyz="0 0 0"
+        rpy="0 0 0" />
+      <geometry>
+        <mesh
+          filename="package://nick_bot/meshes/link_4.STL" />
       </geometry>
     </collision>
@@ -261,6 +258,5 @@
       upper="3.1415"
       effort="300"
-      velocity="4" />
-    <dynamics damping="${joint_damping}"/>
+      velocity="4.0" />
   </joint>
   <link
@@ -271,34 +267,29 @@
         rpy="0 0 0" />
       <mass
-        value="0.049088" />
-      <inertia
-        ixx="1.0527E-05"
-        ixy="1.4724E-09"
-        ixz="-5.9687E-11"
-        iyy="1.3447E-05"
-        iyz="-1.1209E-06"
-        izz="1.7793E-05" />
-    </inertial>
-    <visual>
-      <origin
-        xyz="0 0 0"
-        rpy="0 0 0" />
-      <geometry>
-        <mesh
-          filename="package://nick_bot_1/meshes/link_5.STL" />
-      </geometry>
-      <material
-        name="">
-        <color
-          rgba="0.79216 0.81961 0.93333 1" />
-      </material>
-    </visual>
-    <collision>
-      <origin
-        xyz="0 0 0"
-        rpy="0 0 0" />
-      <geometry>
-        <mesh
-          filename="package://nick_bot_1/meshes/link_5.STL" />
+        value="0.05" />
+      <inertia ixx="0.0001" ixy="0.000"  ixz="0.000"
+         iyy="0.0001" iyz="0.000"
+         izz="0.0001"/>
+    </inertial>
+    <visual>
+      <origin
+        xyz="0 0 0"
+        rpy="0 0 0" />
+      <geometry>
+        <mesh
+          filename="package://nick_bot/meshes/link_5.STL" />
+      </geometry>
+      <material name="">
+        <color
+          rgba="0.79216 0.81961 0.93333 1" />
+      </material>
+    </visual>
+    <collision>
+      <origin
+        xyz="0 0 0"
+        rpy="0 0 0" />
+      <geometry>
+        <mesh
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
File: src/nick_bot/description/robot_core.xacro (robot description, xacro)
@@ -12,5 +12,5 @@
     <inertial>
       <origin
-        xyz="0 0 2"
+        xyz="-0.00522413960660934 1.01612793732535E-06 0.0266388152879452"
         rpy="0 0 0" />
       <mass
@@ -31,5 +31,5 @@
         name="">
         <color
-          rgba="0.79216 0.81961 0.93333 1" />
+          rgba="0.792156862745098 0.819607843137255 0.933333333333333 1" />
       </material>
     </visual>
@@ -48,5 +48,5 @@
     <inertial>
       <origin
-        xyz="0.0061634 0.0010038 0.060589"
+        xyz="0.00616337962890819 0.00100379018116143 0.0605890124959618"
         rpy="0 0 0" />
       <mass
@@ -67,5 +67,5 @@
         name="">
         <color
-          rgba="0.79216 0.81961 0.93333 1" />
+          rgba="0.792156862745098 0.819607843137255 0.933333333333333 1" />
       </material>
     </visual>
@@ -82,8 +82,8 @@
   <joint
     name="joint_1"
-    type="fixed">
+    type="revolute">
     <origin
       xyz="0 0 0.064087"
-      rpy="0.017453 0 -0.0098054" />
+      rpy="0.017453 0 -1.5621" />
     <parent
       link="base_link" />
@@ -91,10 +91,10 @@
       link="link_1" />
     <axis
-      xyz="0 0.017452 0.99985" />
-    <limit
-      lower="-2.7"
-      upper="2.7"
-      effort="300.0"
-      velocity="4.0" />
+      xyz="0 -0.017452 -0.99985" />
+    <limit
+      lower="-1.75"
+      upper="1.75"
+      effort="0"
+      velocity="0" />
   </joint>
   <link
@@ -102,5 +102,5 @@
     <inertial>
       <origin
-        xyz="-0.03205 0.0005952 0.018073"
+        xyz="-0.0320499775068787 0.000595202453078758 0.018073123575994"
         rpy="0 0 0" />
       <mass
@@ -121,5 +121,5 @@
         name="">
         <color
-          rgba="0.79216 0.81961 0.93333 1" />
+          rgba="0.792156862745098 0.819607843137255 0.933333333333333 1" />
       </material>
     </visual>
@@ -136,8 +136,8 @@
   <joint
     name="joint_2"
-    type="fixed">
+    type="revolute">
     <origin
       xyz="0 0.0024593 0.14089"
-      rpy="1.4125 -0.0087445 -0.0071993" />
+      rpy="1.4835 -0.0088311 -0.0078131" />
     <parent
       link="link_1" />
@@ -145,10 +145,10 @@
       link="link_2" />
     <axis
-      xyz="0.99996 -0.0087252 0.0001523" />
-    <limit
-      lower="-3.5"
-      upper="0.6"
-      effort="300"
-      velocity="4.0" />
+      xyz="-0.99996 0.0087252 -0.0001523" />
+    <limit
+      lower="-0.6"
+      upper="3.6"
+      effort="0"
+      velocity="0" />
   </joint>
   <link
@@ -156,5 +156,5 @@
     <inertial>
       <origin
-        xyz="-0.014774 0.00011596 -0.0036584"
+        xyz="-0.0147738927835156 0.000115773286870235 -0.00365845437443535"
         rpy="0 0 0" />
       <mass
@@ -175,5 +175,5 @@
         name="">
         <color
-          rgba="0.79216 0.81961 0.93333 1" />
+          rgba="0.792156862745098 0.819607843137255 0.933333333333333 1" />
       </material>
     </visual>
@@ -190,8 +190,8 @@
   <joint
     name="joint_3"
-    type="fixed">
+    type="revolute">
     <origin
       xyz="0 0.0019372 0.11098"
-      rpy="1.6508 -0.0088619 -0.009271" />
+      rpy="-1.9199 0.0079947 -0.011853" />
     <parent
       link="link_2" />
@@ -201,8 +201,8 @@
       xyz="-0.99996 0.0087252 -0.0001523" />
     <limit
-      lower="-0.7"
-      upper="4"
-      effort="200"
-      velocity="4.0" />
+      lower="-4.2"
+      upper="0"
+      effort="0"
+      velocity="0" />
   </joint>
   <link
@@ -210,5 +210,5 @@
     <inertial>
       <origin
-        xyz="0.00044646 0.0013719 0.078813"
+        xyz="0.000446439621704181 0.00137190367562623 0.0788129649196884"
         rpy="0 0 0" />
       <mass
@@ -229,5 +229,5 @@
         name="">
         <color
-          rgba="0.79216 0.81961 0.93333 1" />
+          rgba="0.792156862745098 0.819607843137255 0.933333333333333 1" />
       </material>
     </visual>
@@ -244,8 +244,8 @@
   <joint
     name="joint_4"
-    type="fixed">
+    type="revolute">
     <origin
       xyz="0 0 0"
-      rpy="0.015346 0.017326 1.4497" />
+      rpy="0.017453 -0.017453 -1.5708" />
     <parent
       link="link_3" />
@@ -255,8 +255,8 @@
       xyz="0 -0.017452 -0.99985" />
     <limit
-      lower="-3.1415"
-      upper="3.1415"
-      effort="300"
-      velocity="4.0" />
+      lower="-1.5"
+      upper="2"
+      effort="0"
+      velocity="0" />
   </joint>
   <link
@@ -264,5 +264,5 @@
     <inertial>
       <origin
-        xyz="1.3718E-06 -0.011218 0.0025865"
+        xyz="1.37814036968442E-06 -0.0112175744982041 0.00258648216033591"
         rpy="0 0 0" />
       <mass
@@ -280,7 +280,8 @@
           filename="package://nick_bot/meshes/link_5.STL" />
       </geometry>
-      <material name="">
-        <color
-          rgba="0.79216 0.81961 0.93333 1" />
+      <material
+        name="">
+        <color
+          rgba="0.792156862745098 0.819607843137255 0.933333333333333 1" />
       </material>
     </visual>
@@ -297,8 +298,8 @@
   <joint
     name="joint_5"
-    type="fixed">
+    type="revolute">
     <origin
       xyz="0 0.0032854 0.18822"
-      rpy="-1.909 0.0001523 3.1329" />
+      rpy="-0.017453 -0.0001523 -0.0087253" />
     <parent
       link="link_4" />
@@ -306,10 +307,10 @@
       link="link_5" />
     <axis
-      xyz="1 0 0" />
-    <limit
-      lower="0"
-      upper="4"
-      effort="200"
-      velocity="4.0" />
+      xyz="-1 0 0" />
+    <limit
+      lower="-2.35"
+      upper="2.35"
+      effort="0"
+      velocity="0" />
   </joint>
   <link
@@ -317,5 +318,5 @@
     <inertial>
       <origin
-        xyz="1.2663E-08 0.020431 2.0602E-08"
+        xyz="-1.66377830262965E-08 0.0204269190545232 3.44363878523879E-08"
         rpy="0 0 0" />
       <mass
@@ -336,5 +337,5 @@
         name="">
         <color
-          rgba="0.79216 0.81961 0.93333 1" />
+          rgba="0.792156862745098 0.819607843137255 0.933333333333333 1" />
       </material>
     </visual>
@@ -351,8 +352,8 @@
   <joint
     name="joint_6"
-    type="revolute">
+    type="continuous">
     <origin
       xyz="0 0 0"
-      rpy="1.5708 0 1.6504" />
+      rpy="1.5708 0 2.2137" />
     <parent
       link="link_5" />
@@ -361,9 +362,4 @@
     <axis
       xyz="0 -1 0" />
-    <limit
-      lower="-3.1415"
-      upper="3.1415"
-      effort="200"
-      velocity="4.0" />
   </joint>
   <gazebo reference="link_1">

File: src/nick_bot/description/ros2_control.xacro (robot description, xacro)
@@ -1,5 +1,5 @@
 <?xml version="1.0"?>
 <robot xmlns:xacro="http://www.ros.org/wiki/xacro">
- <ros2_control name="RealRobot" type="system">
+ <ros2_control name="RealRobotServos" type="system">
    <hardware>
      <plugin>dynamixel_hardware/DynamixelHardware</plugin>
@@ -8,12 +8,60 @@
        <!-- <param name="use_dummy">true</param> -->
   </hardware>
-    <joint name="joint_6">
+	<joint name="joint_5">
+      <param name="id">2</param>
+  	  <command_interface name="position"/>
+  	  <state_interface name="position">
+  	    <param name="initial_value">0</param>
+  	   </state_interface>
+  	  <state_interface name="velocity"/>
+  	</joint>
+  	<joint name="joint_6">
+      <param name="id">3</param>
+  	  <command_interface name="position"/>
+  	  <state_interface name="position">
+  	    <param name="initial_value">0</param>
+  	   </state_interface>
+  	  <state_interface name="velocity"/>
+  	</joint>
+  	<joint name="joint_4">
       <param name="id">1</param>
   	  <command_interface name="position"/>
   	  <state_interface name="position">
-  	    <param name="initial_value">-1.32996</param>
+  	    <param name="initial_value">0</param>
   	   </state_interface>
   	  <state_interface name="velocity"/>
   	</joint>
+  </ros2_control>
+  <ros2_control name="RealRobotSteppers" type="system">
+   <hardware>
+     <plugin>stepper_interface/StepperInterface</plugin>
+       <param name="device_port">/tmp/ttyV1</param>
+       <param name="baud_rate">1000000</param>
+       <param name="timeout">1000</param>
+  </hardware>
+    <joint name="joint_1">
+        <param name="name">base</param>
+        <command_interface name="position"/>
+  	<state_interface name="position">
+  	  <param name="initial_value">0</param>
+  	</state_interface>
+  	<!-- <state_interface name="velocity"/> -->
+     </joint>
+     <joint name="joint_2">
+        <param name="name">shoulder</param>
+        <command_interface name="position"/>
+  	<state_interface name="position">
+  	  <param name="initial_value">0</param>
+  	</state_interface>
+  	<!-- <state_interface name="velocity"/> -->
+     </joint>
+     <joint name="joint_3">
+        <param name="name">elbow</param>
+        <command_interface name="position"/>
+  	<state_interface name="position">
+  	  <param name="initial_value">0</param>
+  	</state_interface>
+  	<!-- <state_interface name="velocity"/> -->
+     </joint>
   </ros2_control>
   <transmission name="link_1_trans">

File: src/nick_bot/urdf/nick_bot.urdf (robot description, URDF)
Before this commit: robot nick_bot, 8 links, 7 joints
Links:
- link base_link: mass 0.51245 -> 0.05
- link end_effector: mass 0.01147 -> 0.05
- link link_1: mass 0.28024 -> 0.05
- link link_2: mass 0.29393 -> 0.05
- link link_3: mass 0.085607 -> 0.05
- link link_4: mass 0.15698 -> 0.05
- link link_5: mass 0.049088 -> 0.05
Joints:
- joint base_joint: origin xyz=0.0 0.0 0.0 rpy=0 0 0 -> xyz=0.0 0.0 0.3 rpy=0 0 0
- joint joint_1: axis 0 0.017452 0.99985 -> 0 -0.017452 -0.99985; limit lower=-2.7 upper=2.7 effort=300.0 velocity=4.0 -> lower=-1.75 upper=1.75 effort=0 velocity=0; origin xyz=0 0 0.064087 rpy=0.017453 0 -0.0098054 -> xyz=0 0 0.064087 rpy=0.017453 0 -1.5621
- joint joint_2: axis 0.99996 -0.0087252 0.0001523 -> -0.99996 0.0087252 -0.0001523; limit lower=-3.5 upper=0.6 effort=300 velocity=4.0 -> lower=-0.6 upper=3.6 effort=0 velocity=0; origin xyz=0 0.0024593 0.14089 rpy=1.4125 -0.0087445 -0.0071993 -> xyz=0 0.0024593 0.14089 rpy=1.4835 -0.0088311 -0.0078131
- joint joint_3: limit lower=-0.7 upper=4 effort=200 velocity=4.0 -> lower=-4.2 upper=0 effort=0 velocity=0; origin xyz=0 0.0019372 0.11098 rpy=1.6508 -0.0088619 -0.009271 -> xyz=0 0.0019372 0.11098 rpy=-1.9199 0.0079947 -0.011853
- joint joint_4: limit lower=-3.1415 upper=3.1415 effort=300 velocity=4.0 -> lower=-1.5 upper=2 effort=0 velocity=0; origin xyz=0 0 0 rpy=0.015346 0.017326 1.4497 -> xyz=0 0 0 rpy=0.017453 -0.017453 -1.5708
- joint joint_5: axis 1 0 0 -> -1 0 0; limit lower=0 upper=4 effort=200 velocity=4.0 -> lower=-2.35 upper=2.35 effort=0 velocity=0; origin xyz=0 0.0032854 0.18822 rpy=-1.909 0.0001523 3.1329 -> xyz=0 0.0032854 0.18822 rpy=-0.017453 -0.0001523 -0.0087253
- joint joint_6: limit lower=-3.1415 upper=3.1415 effort=200 velocity=4.0 -> (none); origin xyz=0 0 0 rpy=1.5708 0 1.6504 -> xyz=0 0 0 rpy=1.5708 0 2.2137; type revolute -> continuous

File: src/nick_bot_moveit_config/config/nick_bot.ros2_control.xacro (robot description, xacro)
@@ -8,8 +8,8 @@
                 <plugin>gazebo_ros2_control/GazeboSystem</plugin>
             </hardware>
-            <joint name="joint_6">
+            <joint name="joint_4">
                 <command_interface name="position"/>
                 <state_interface name="position">
-                  <param name="initial_value">${initial_positions['joint_6']}</param>
+                  <param name="initial_value">${initial_positions['joint_4']}</param>
                 </state_interface>
                 <state_interface name="velocity"/>
