Commit message: commti real robot launch

File: src/nick_bot/description/ros2_control.xacro (robot description, xacro)
@@ -8,5 +8,13 @@
        <!-- <param name="use_dummy">true</param> -->
   </hardware>
-	<joint name="joint_5">
+    <joint name="joint_4">
+      <param name="id">1</param>
+  	  <command_interface name="position"/>
+  	  <state_interface name="position">
+  	    <param name="initial_value">0</param>
+  	   </state_interface>
+  	  <state_interface name="velocity"/>
+  	</joint>
+  	<joint name="joint_5">
       <param name="id">2</param>
   	  <command_interface name="position"/>
@@ -24,17 +32,9 @@
   	  <state_interface name="velocity"/>
   	</joint>
-  	<joint name="joint_4">
-      <param name="id">1</param>
-  	  <command_interface name="position"/>
-  	  <state_interface name="position">
-  	    <param name="initial_value">0</param>
-  	   </state_interface>
-  	  <state_interface name="velocity"/>
-  	</joint>
   </ros2_control>
   <ros2_control name="RealRobotSteppers" type="system">
    <hardware>
      <plugin>stepper_interface/StepperInterface</plugin>
-       <param name="device_port">/tmp/ttyV1</param>
+       <param name="device_port">/dev/ttyACM0</param>
        <param name="baud_rate">1000000</param>
        <param name="timeout">1000</param>
