Commit message: workign with one dynamixel

File: src/nick_bot/description/robot_core.xacro (robot description, xacro)
@@ -82,5 +82,5 @@
   <joint
     name="joint_1"
-    type="revolute">
+    type="fixed">
     <origin
       xyz="0 0 0.064087"
@@ -136,5 +136,5 @@
   <joint
     name="joint_2"
-    type="revolute">
+    type="fixed">
     <origin
       xyz="0 0.0024593 0.14089"
@@ -190,5 +190,5 @@
   <joint
     name="joint_3"
-    type="revolute">
+    type="fixed">
     <origin
       xyz="0 0.0019372 0.11098"
@@ -244,5 +244,5 @@
   <joint
     name="joint_4"
-    type="revolute">
+    type="fixed">
     <origin
       xyz="0 0 0"
@@ -297,5 +297,5 @@
   <joint
     name="joint_5"
-    type="revolute">
+    type="fixed">
     <origin
       xyz="0 0.0032854 0.18822"

File: src/nick_bot/description/ros2_controlGAZEBO.xacro (robot description, xacro)
@@ -1,13 +1,49 @@
 <?xml version="1.0"?>
 <robot xmlns:xacro="http://www.ros.org/wiki/xacro">
- <ros2_control name="RealRobot" type="system">
-   <hardware>
-     <plugin>dynamixel_hardware/DynamixelHardware</plugin>
-       <param name="usb_port">/dev/ttyUSB1</param>
-       <param name="baud_rate">1000000</param>
-       <!-- <param name="use_dummy">true</param> -->
-  </hardware>
-    <joint name="joint_6">
-      <param name="id">1</param>
+    <gazebo>
+        <plugin name="gazebo_ros2_control" filename="libgazebo_ros2_control.so">
+            <parameters> $(find nick_bot)/config/nickbot_controllers.yaml</parameters>
+        </plugin>
+    </gazebo>
+  <ros2_control name="GazeboSystem" type="system">
+  	<hardware>
+  	  <plugin>gazebo_ros2_control/GazeboSystem</plugin>
+  	</hardware>
+  	<joint name="joint_1">
+  	  <command_interface name="position"/>
+  	  <state_interface name="position">
+  	    <param name="initial_value">0.0</param>
+  	   </state_interface>
+  	   <state_interface name="velocity"/>
+  	</joint>
+  	<joint name="joint_2">
+  	  <command_interface name="position"/>
+  	  <state_interface name="position">
+  	    <param name="initial_value">0.0</param>
+  	   </state_interface>
+  	   <state_interface name="velocity"/>
+  	</joint>
+  	<joint name="joint_3">
+  	  <command_interface name="position"/>
+  	  <state_interface name="position">
+  	    <param name="initial_value">0.0</param>
+  	   </state_interface>
+  	   <state_interface name="velocity"/>
+  	</joint>
+  	<joint name="joint_4">
+  	  <command_interface name="position"/>
+  	  <state_interface name="position">
+  	    <param name="initial_value">0.0</param>
+  	   </state_interface>
+  	   <state_interface name="velocity"/>
+  	</joint>
+  	<joint name="joint_5">
+  	  <command_interface name="position"/>
+  	  <state_interface name="position">
+  	    <param name="initial_value">0.0</param>
+  	   </state_interface>
+  	   <state_interface name="velocity"/>
+  	</joint>
+  	<joint name="joint_6">
   	  <command_interface name="position"/>
   	  <state_interface name="position">

File: src/nick_bot_moveit_config/config/nick_bot.ros2_control.xacro (robot description, xacro)
@@ -8,39 +8,4 @@
                 <plugin>gazebo_ros2_control/GazeboSystem</plugin>
             </hardware>
-            <joint name="joint_1">
-                <command_interface name="position"/>
-                <state_interface name="position">
-                  <param name="initial_value">${initial_positions['joint_1']}</param>
-                </state_interface>
-                <state_interface name="velocity"/>
-            </joint>
-            <joint name="joint_2">
-                <command_interface name="position"/>
-                <state_interface name="position">
-                  <param name="initial_value">${initial_positions['joint_2']}</param>
-                </state_interface>
-                <state_interface name="velocity"/>
-            </joint>
-            <joint name="joint_3">
-                <command_interface name="position"/>
-                <state_interface name="position">
-                  <param name="initial_value">${initial_positions['joint_3']}</param>
-                </state_interface>
-                <state_interface name="velocity"/>
-            </joint>
-            <joint name="joint_4">
-                <command_interface name="position"/>
-                <state_interface name="position">
-                  <param name="initial_value">${initial_positions['joint_4']}</param>
-                </state_interface>
-                <state_interface name="velocity"/>
-            </joint>
-            <joint name="joint_5">
-                <command_interface name="position"/>
-                <state_interface name="position">
-                  <param name="initial_value">${initial_positions['joint_5']}</param>
-                </state_interface>
-                <state_interface name="velocity"/>
-            </joint>
             <joint name="joint_6">
                 <command_interface name="position"/>

Commit message: update hardware (mainly)

File: src/nick_bot/description/robot_core.xacro (robot description, xacro)
@@ -255,6 +255,6 @@
       xyz="0 -0.017452 -0.99985" />
     <limit
-      lower="-1.5"
-      upper="2"
+      lower="-4.7"
+      upper="4.7"
       effort="0"
       velocity="0" />

File: src/nick_bot/description/ros2_control.xacro (robot description, xacro)
@@ -9,5 +9,5 @@
   </hardware>
     <joint name="joint_4">
-      <param name="id">1</param>
+      <param name="id">3</param>
   	  <command_interface name="position"/>
   	  <state_interface name="position">
@@ -25,5 +25,5 @@
   	</joint>
   	<joint name="joint_6">
-      <param name="id">3</param>
+      <param name="id">1</param>
   	  <command_interface name="position"/>
   	  <state_interface name="position">

File: src/nick_bot/urdf/nick_bot.urdf (robot description, URDF)
Before this commit: robot nick_bot, 8 links, 7 joints
Joints:
- joint joint_4: limit lower=-1.5 upper=2 effort=0 velocity=0 -> lower=-4.7 upper=4.7 effort=0 velocity=0
